Commit message: basic gazebo intigration , next step ros2 control with gazebo

File: src/panda_ros_simulation/urdf/gripper.urdf.xacro (robot description, xacro)
@@ -15,42 +15,28 @@
             joint_type="fixed" joint_origin_xyz="0 0 0"
             joint_origin_rpy="0 0 0" />
-        <xacro:property name="joint_finger1_origin_xyz" value="0 0 0.0584" />
-        <xacro:property name="joint_finger1_origin_rpy" value="0 0 0" />
-        <xacro:property name="joint_finger1_axis_xyz" value="0 1 0" />
-        <xacro:property name="joint_finger1_lower_limit" value="0" />
-        <xacro:property name="joint_finger1_upper_limit" value="0.04" />
-        <xacro:property name="joint_finger1_velocity_limit" value="0.2" />
-        <xacro:property name="joint_finger1_torque_limit" value="20" />
-        <xacro:property name="joint_finger1_damping" value="3.0" />
-        <xacro:property name="joint_finger1_friction" value="0.4" />
-        <xacro:property name="joint_finger2_origin_xyz" value="0 0 0.0584" />
-        <xacro:property name="joint_finger2_origin_rpy" value="0 0 3.14" />
-        <xacro:property name="joint_finger2_axis_xyz" value="0 -1 0" />
-        <xacro:property name="joint_finger2_lower_limit" value="-0.04" />
-        <xacro:property name="joint_finger2_upper_limit" value="0" />
-        <xacro:property name="joint_finger2_velocity_limit" value="0.2" />
-        <xacro:property name="joint_finger2_torque_limit" value="20" />
-        <xacro:property name="joint_finger2_damping" value="3.0" />
-        <xacro:property name="joint_finger2_friction" value="0.4" />
+        <!-- ... (finger_joint1 definition is unchanged) ... -->
         <xacro:panda_joint parent="${gripper_hand_link_name}" child="${finger_link1_name}"
             joint_name="finger_joint1"
-            joint_type="prismatic" joint_origin_xyz="${joint_finger1_origin_xyz}"
-            joint_origin_rpy="${joint_finger1_origin_rpy}"
-            joint_axis_xyz="${joint_finger1_axis_xyz}"
-            joint_lower_limit="${joint_finger1_lower_limit}"
-            joint_upper_limit="${joint_finger1_upper_limit}"
-            joint_velocity_limit="${joint_finger1_velocity_limit}"
-            joint_torque_limit="${joint_finger1_torque_limit}"
-            joint_damping="${joint_finger1_damping}" joint_friction="${joint_finger1_friction}" />
+            joint_type="prismatic" joint_origin_xyz="0 0 0.0584"
+            joint_origin_rpy="0 0 0"
+            joint_axis_xyz="0 1 0"
+            joint_lower_limit="0"
+            joint_upper_limit="0.04"
+            joint_velocity_limit="0.2"
+            joint_torque_limit="20"
+            joint_damping="3.0" joint_friction="0.4" />
+        <!-- The mimic tag is correctly placed inside the macro call for finger_joint2 -->
         <xacro:panda_joint parent="${gripper_hand_link_name}" child="${finger_link2_name}"
             joint_name="finger_joint2"
-            joint_type="prismatic" joint_origin_xyz="${joint_finger2_origin_xyz}"
-            joint_origin_rpy="${joint_finger2_origin_rpy}"
-            joint_axis_xyz="${joint_finger2_axis_xyz}"
-            joint_lower_limit="${joint_finger2_lower_limit}"
-            joint_upper_limit="${joint_finger2_upper_limit}"
-            joint_velocity_limit="${joint_finger2_velocity_limit}"
-            joint_torque_limit="${joint_finger2_torque_limit}"
-            joint_damping="${joint_finger2_damping}" joint_friction="${joint_finger2_friction}" />
+            joint_type="prismatic" joint_origin_xyz="0 0 0.0584"
+            joint_origin_rpy="0 0 3.14"
+            joint_axis_xyz="0 -1 0"
+            joint_lower_limit="-0.04"
+            joint_upper_limit="0"
+            joint_velocity_limit="0.2"
+            joint_torque_limit="20"
+            joint_damping="3.0" joint_friction="0.4">
+            <!-- <mimic joint="finger_joint1" multiplier="-1" offset="0" /> -->
+        </xacro:panda_joint>
     </xacro:macro>
 </robot>

File: src/panda_ros_simulation/urdf/macros.urdf.xacro (robot description, xacro)
@@ -54,4 +54,20 @@
                 <dynamics damping="${joint_damping}" friction="${joint_friction}" />
             </xacro:unless>
+            <xacro:if value="${joint_name == 'finger_joint1'}">
+                <gazebo>
+                    <joint name="finger_joint1">
+                        <position>0.01</position>
+                    </joint>
+                </gazebo>
+            </xacro:if>
+            <xacro:if value="${joint_name == 'finger_joint2'}">
+                <mimic joint="finger_joint1" multiplier="-1"
+                    offset="0" />
+                <gazebo>
+                    <joint name="finger_joint2">
+                        <position>-0.01</position>
+                    </joint>
+                </gazebo>
+            </xacro:if>
         </joint>
         <xacro:unless value="${joint_type == 'fixed'}">

File: src/panda_ros_simulation/urdf/panda.urdf.xacro (robot description, xacro)
@@ -1,19 +1,19 @@
 <?xml version="1.0"?>
 <robot name="franka_panda" xmlns:xacro="http://www.ros.org/wiki/xacro">
-  <xacro:property name="mesh_pkg_visual" value="package://panda_ros_simulation/meshes/visual" />
-  <xacro:property name="mesh_pkg_collision" value="package://panda_ros_simulation/meshes/collision" />
+  <xacro:property name="mesh_pkg_visual" value="/home/akhil/panda_ros_simulation/install/panda_ros_simulation/share/panda_ros_simulation/meshes/visual" />
+  <xacro:property name="mesh_pkg_collision" value="/home/akhil/panda_ros_simulation/install/panda_ros_simulation/share/panda_ros_simulation/meshes/collision" />
   <xacro:property name="mesh_pkg_description" value="package://panda_ros_simulation/urdf" />
   <xacro:include filename="$(find panda_ros_simulation)/urdf/macros.urdf.xacro" />
   <xacro:include filename="$(find panda_ros_simulation)/urdf/props.urdf.xacro" />
   <xacro:include filename="$(find panda_ros_simulation)/urdf/gripper.urdf.xacro" />
-    <material name="panda_gray">
-        <color rgba="0.7 0.7 0.7 1" />
-    </material>
-    <material name="panda_dark">
-        <color rgba="0.2 0.2 0.2 1" />
-    </material>
-    <material name="panda_white">
-        <color rgba="0.95 0.95 0.95 1" />
-    </material>
+  <material name="panda_gray">
+    <color rgba="0.7 0.7 0.7 1" />
+  </material>
+  <material name="panda_dark">
+    <color rgba="0.2 0.2 0.2 1" />
+  </material>
+  <material name="panda_white">
+    <color rgba="0.95 0.95 0.95 1" />
+  </material>
   <!-- <link name="world" /> -->
   <link name="base_link" />
@@ -184,9 +184,9 @@
     gazebo_preserve_fixed_joint="true"
   /> -->
-<joint name="panda_link7_to_link8" type="fixed">
-  <parent link="panda_link7" />
-  <child link="panda_link8" />
-  <origin xyz="${wrist_origin_xyz}" rpy="${wrist_origin_rpy}" />
-</joint>
+  <joint name="panda_link7_to_link8" type="fixed">
+    <parent link="panda_link7" />
+    <child link="panda_link8" />
+    <origin xyz="${wrist_origin_xyz}" rpy="${wrist_origin_rpy}" />
+  </joint>
   <!-- **********End of kinamatic chain***** -->
   <!--####################################Start
@@ -197,5 +197,5 @@
     finger_link2_name="panda_rightfinger"
   />
-  <ros2_control name="PandaSystem" type="system">
+  <!-- <ros2_control name="PandaSystem" type="system">
     <hardware>
       <plugin>gazebo_ros2_control/GazeboSystem</plugin>
@@ -261,4 +261,26 @@
       <robot_param_node>robot_state_publisher</robot_param_node>
     </plugin>
+  </gazebo> -->
+  <gazebo>
+    <plugin name="gazebo_ros_joint_state_publisher"
+      filename="libgazebo_ros_joint_state_publisher.so">
+      <update_rate>20</update_rate>
+      <joint_name>panda_joint1</joint_name>
+      <joint_name>panda_joint2</joint_name>
+      <joint_name>panda_joint3</joint_name>
+      <joint_name>panda_joint4</joint_name>
+      <joint_name>panda_joint5</joint_name>
+      <joint_name>panda_joint6</joint_name>
+      <joint_name>panda_joint7</joint_name>
+      <joint_name>finger_joint1</joint_name>
+      <joint_name>finger_joint2</joint_name>
+    </plugin>
+    <!-- <plugin name="gazebo_ros_init"
+      filename="libgazebo_ros_init.so">
+      <parameters>
+        <joint_name>finger_joint1</joint_name>
+        <initial_position>0.02</initial_position>
+      </parameters>
+    </plugin> -->
   </gazebo>
 </robot>
