Commit message: final, gazebo loading the model properly

File: src/panda_ros_simulation/urdf/macros.urdf.xacro (robot description, xacro)
@@ -17,4 +17,7 @@
             <xacro:panda_inertial mesh="${imesh}" mesh_offset_rpy="0 0 0" />
         </link>
+        <gazebo reference="${lname}">
+        <material>Gazebo/Grey</material>
+    </gazebo>
     </xacro:macro>
     <!-- Macro for joining the links -->

File: src/panda_ros_simulation/urdf/panda.urdf.xacro (robot description, xacro)
@@ -1,6 +1,6 @@
 <?xml version="1.0"?>
 <robot name="franka_panda" xmlns:xacro="http://www.ros.org/wiki/xacro">
-  <xacro:property name="mesh_pkg_visual" value="/home/akhil/panda_ros_simulation/install/panda_ros_simulation/share/panda_ros_simulation/meshes/visual" />
-  <xacro:property name="mesh_pkg_collision" value="/home/akhil/panda_ros_simulation/install/panda_ros_simulation/share/panda_ros_simulation/meshes/collision" />
+  <xacro:property name="mesh_pkg_visual" value="file:///home/akhil/panda_ros_simulation/install/panda_ros_simulation/share/panda_ros_simulation/meshes/visual" />
+  <xacro:property name="mesh_pkg_collision" value="file:///home/akhil/panda_ros_simulation/install/panda_ros_simulation/share/panda_ros_simulation/meshes/collision" />
   <xacro:property name="mesh_pkg_description" value="package://panda_ros_simulation/urdf" />
   <xacro:include filename="$(find panda_ros_simulation)/urdf/macros.urdf.xacro" />
@@ -16,11 +16,11 @@
     <color rgba="0.95 0.95 0.95 1" />
   </material>
-  <!-- <link name="world" /> -->
+  <link name="world" />
   <link name="base_link" />
-  <!-- <joint name="world_to_base" type="fixed">
+  <joint name="world_to_base" type="fixed">
     <parent link="world" />
     <child link="base_link" />
     <origin xyz="0 0 0" rpy="0 0 0" />
-  </joint> -->
+  </joint>
   <xacro:panda_link lname="panda_link0" vmesh="${mesh_pkg_visual}/link0.dae"
     cmesh="${mesh_pkg_collision}/link0.stl" imesh="${link0_mesh}" color="panda_dark" />
@@ -177,11 +177,4 @@
   <xacro:property name="wrist_origin_xyz" value="0 0 0.107" />
   <xacro:property name="wrist_origin_rpy" value="0 0 ${-pi/4}" />
-  <!-- <xacro:panda_virtual_link
-    parent="panda_link7"
-    link_name="panda_link8V"
-    joint_origin_xyz="${wrist_origin_xyz}"
-    joint_origin_rpy="${wrist_origin_rpy}"
-    gazebo_preserve_fixed_joint="true"
-  /> -->
   <joint name="panda_link7_to_link8" type="fixed">
     <parent link="panda_link7" />
@@ -276,11 +269,4 @@
       <joint_name>finger_joint2</joint_name>
     </plugin>
-    <!-- <plugin name="gazebo_ros_init"
-      filename="libgazebo_ros_init.so">
-      <parameters>
-        <joint_name>finger_joint1</joint_name>
-        <initial_position>0.02</initial_position>
-      </parameters>
-    </plugin> -->
   </gazebo>
 </robot>

Commit message: movit2

File: src/panda_ros_simulation/urdf/macros.urdf.xacro (robot description, xacro)
@@ -2,5 +2,5 @@
 <robot xmlns:xacro="http://www.ros.org/wiki/xacro">
     <!-- Macro for creating links -->
-    <xacro:macro name="panda_link" params="lname vmesh cmesh imesh color">
+    <xacro:macro name="panda_link" params="lname vmesh cmesh imesh color rgba_val">
         <link name="${lname}">
             <visual>
@@ -18,6 +18,11 @@
         </link>
         <gazebo reference="${lname}">
-        <material>Gazebo/Grey</material>
-    </gazebo>
+            <material>
+               ${rgba_val}
+            </material>
+        </gazebo>
+       <!-- <gazebo reference="${lname}">
+        <material>Gazebo/White</material>
+    </gazebo> -->
     </xacro:macro>
     <!-- Macro for joining the links -->

File: src/panda_ros_simulation/urdf/panda.urdf.xacro (robot description, xacro)
@@ -18,4 +18,8 @@
     <color rgba="0.95 0.95 0.95 1" />
   </material>
+  <xacro:property name="panda_gray" value="Gazebo/Grey" />
+  <xacro:property name="panda_dark" value="Gazebo/Red" />
+  <xacro:property name="panda_white" value="Gazebo/White" />
+  <xacro:property name="panda_green" value="Gazebo/Green" />
   <link name="world" />
   <link name="base_link" />
@@ -26,25 +30,25 @@
   </joint>
   <xacro:panda_link lname="panda_link0" vmesh="${mesh_pkg_visual}/link0.dae"
-    cmesh="${mesh_pkg_collision}/link0.stl" imesh="${link0_mesh}" color="panda_dark" />
+    cmesh="${mesh_pkg_collision}/link0.stl" imesh="${link0_mesh}" color="panda_dark" rgba_val="${panda_dark}"/>
   <xacro:panda_link lname="panda_link1" vmesh="${mesh_pkg_visual}/link1.dae"
-    cmesh="${mesh_pkg_collision}/link1.stl" imesh="${link1_mesh}" color="panda_gray" />
+    cmesh="${mesh_pkg_collision}/link1.stl" imesh="${link1_mesh}" color="panda_gray" rgba_val= "${panda_gray}"/>
   <xacro:panda_link lname="panda_link2" vmesh="${mesh_pkg_visual}/link2.dae"
-    cmesh="${mesh_pkg_collision}/link2.stl" imesh="${link2_mesh}" color="panda_white" />
+    cmesh="${mesh_pkg_collision}/link2.stl" imesh="${link2_mesh}" color="panda_white" rgba_val="${panda_white}"/>
   <xacro:panda_link lname="panda_link3" vmesh="${mesh_pkg_visual}/link3.dae"
-    cmesh="${mesh_pkg_collision}/link3.stl" imesh="${link3_mesh}" color="panda_gray" />
+    cmesh="${mesh_pkg_collision}/link3.stl" imesh="${link3_mesh}" color="panda_gray" rgba_val="${panda_gray}"/>
   <xacro:panda_link lname="panda_link4" vmesh="${mesh_pkg_visual}/link4.dae"
-    cmesh="${mesh_pkg_collision}/link4.stl" imesh="${link4_mesh}" color="panda_white" />
+    cmesh="${mesh_pkg_collision}/link4.stl" imesh="${link4_mesh}" color="panda_white" rgba_val="${panda_white}"/>
   <xacro:panda_link lname="panda_link5" vmesh="${mesh_pkg_visual}/link5.dae"
-    cmesh="${mesh_pkg_collision}/link5.stl" imesh="${link5_mesh}" color="panda_gray" />
+    cmesh="${mesh_pkg_collision}/link5.stl" imesh="${link5_mesh}" color="panda_gray" rgba_val= "${panda_gray}"/>
   <xacro:panda_link lname="panda_link6" vmesh="${mesh_pkg_visual}/link6.dae"
-    cmesh="${mesh_pkg_collision}/link6.stl" imesh="${link6_mesh}" color="panda_white" />
+    cmesh="${mesh_pkg_collision}/link6.stl" imesh="${link6_mesh}" color="panda_white" rgba_val="${panda_white}" />
   <xacro:panda_link lname="panda_link7" vmesh="${mesh_pkg_visual}/link7.dae"
-    cmesh="${mesh_pkg_collision}/link7.stl" imesh="${link7_mesh}" color="panda_dark" />
+    cmesh="${mesh_pkg_collision}/link7.stl" imesh="${link7_mesh}" color="panda_dark" rgba_val="${panda_dark}"/>
   <xacro:panda_link lname="panda_hand" vmesh="${mesh_pkg_visual}/hand.dae"
-    cmesh="${mesh_pkg_collision}/hand.stl" imesh="${hand_mesh}" color="panda_dark" />
+    cmesh="${mesh_pkg_collision}/hand.stl" imesh="${hand_mesh}" color="panda_dark" rgba_val="${panda_dark}" />
   <xacro:panda_link lname="panda_leftfinger" vmesh="${mesh_pkg_visual}/finger.dae"
-    cmesh="${mesh_pkg_collision}/finger.stl" imesh="${finger_mesh}" color="panda_gray" />
+    cmesh="${mesh_pkg_collision}/finger.stl" imesh="${finger_mesh}" color="panda_gray" rgba_val="${panda_green}"/>
   <xacro:panda_link lname="panda_rightfinger" vmesh="${mesh_pkg_visual}/finger.dae"
-    cmesh="${mesh_pkg_collision}/finger.stl" imesh="${finger_mesh}" color="panda_gray" />
+    cmesh="${mesh_pkg_collision}/finger.stl" imesh="${finger_mesh}" color="panda_gray" rgba_val="${panda_green}"/>
   <link name="panda_link8" />
   <xacro:property name="joint1_origin_xyz" value="0 0 0.333" />
@@ -224,5 +228,5 @@
       <command_interface name="velocity" />
       <state_interface name="position">
-        <param name="initial_value">0.0</param>
+        <param name="initial_value">-1.7</param>
       </state_interface>
       <state_interface name="velocity" />
@@ -232,5 +236,5 @@
       <command_interface name="velocity" />
       <state_interface name="position">
-        <param name="initial_value">0.0</param>
+        <param name="initial_value">-0.7</param>
       </state_interface>
       <state_interface name="velocity" />
