Commit message: Added inertial props

File: src/panda_ros_simulation/urdf/panda.urdf.xacro (robot description, xacro)
@@ -3,8 +3,10 @@
   <xacro:property name="mesh_pkg_visual" value="package://panda_ros_simulation/meshes/visual"/>
   <xacro:property name="mesh_pkg_collision" value="package://panda_ros_simulation/meshes/collision"/>
+  <xacro:property name="mesh_pkg_description" value="package://panda_ros_simulation/urdf"/>
+  <xacro:include filename="$(find panda_ros_simulation)/urdf/props.urdf.xacro"/>
   <material name="panda_gray"><color rgba="0.7 0.7 0.7 1"/></material>
   <material name="panda_dark"><color rgba="0.2 0.2 0.2 1"/></material>
   <material name="panda_white"><color rgba="0.95 0.95 0.95 1"/></material>
-<xacro:macro name="panda_link" params="lname vmesh cmesh color mass ixx iyy izz">
+<xacro:macro name="panda_link" params="lname vmesh cmesh imesh color mass ixx iyy izz">
     <link name="${lname}">
       <visual>
@@ -15,9 +17,5 @@
         <geometry><mesh filename="${cmesh}" scale="1 1 1"/></geometry>
       </collision>
-      <inertial>
-        <origin xyz="0 0 0" rpy="0 0 0"/>
-        <mass value="${mass}"/>
-        <inertia ixx="${ixx}" ixy="0.0" ixz="0.0" iyy="${iyy}" iyz="0.0" izz="${izz}"/>
-      </inertial>
+      <xacro:panda_inertial mesh="${imesh}" mesh_offset_rpy="0 0 0"/>
     </link>
 </xacro:macro>
@@ -29,15 +27,15 @@
     <origin xyz="0 0 0" rpy="0 0 0"/>
   </joint>
-  <xacro:panda_link lname="panda_link0" vmesh="${mesh_pkg_visual}/link0.dae" cmesh="${mesh_pkg_collision}/link0.stl" color="panda_dark" mass="1.0" ixx="0.01" iyy="0.01" izz="0.01"/>
-  <xacro:panda_link lname="panda_link1" vmesh="${mesh_pkg_visual}/link1.dae" cmesh="${mesh_pkg_collision}/link1.stl" color="panda_gray" mass="1.0" ixx="0.01" iyy="0.01" izz="0.01"/>
-  <xacro:panda_link lname="panda_link2" vmesh="${mesh_pkg_visual}/link2.dae" cmesh="${mesh_pkg_collision}/link2.stl" color="panda_white" mass="1.0" ixx="0.01" iyy="0.01" izz="0.01"/>
-  <xacro:panda_link lname="panda_link3" vmesh="${mesh_pkg_visual}/link3.dae" cmesh="${mesh_pkg_collision}/link3.stl" color="panda_gray" mass="1.0" ixx="0.01" iyy="0.01" izz="0.01"/>
-  <xacro:panda_link lname="panda_link4" vmesh="${mesh_pkg_visual}/link4.dae" cmesh="${mesh_pkg_collision}/link4.stl" color="panda_white" mass="1.0" ixx="0.01" iyy="0.01" izz="0.01"/>
-  <xacro:panda_link lname="panda_link5" vmesh="${mesh_pkg_visual}/link5.dae" cmesh="${mesh_pkg_collision}/link5.stl" color="panda_gray" mass="1.0" ixx="0.01" iyy="0.01" izz="0.01"/>
-  <xacro:panda_link lname="panda_link6" vmesh="${mesh_pkg_visual}/link6.dae" cmesh="${mesh_pkg_collision}/link6.stl" color="panda_white" mass="0.8" ixx="0.008" iyy="0.008" izz="0.008"/>
-  <xacro:panda_link lname="panda_link7" vmesh="${mesh_pkg_visual}/link7.dae" cmesh="${mesh_pkg_collision}/link7.stl" color="panda_dark" mass="0.6" ixx="0.006" iyy="0.006" izz="0.006"/>
-  <xacro:panda_link lname="panda_hand" vmesh="${mesh_pkg_visual}/hand.dae" cmesh="${mesh_pkg_collision}/hand.stl" color="panda_dark" mass="0.2" ixx="0.002" iyy="0.002" izz="0.002"/>
-  <xacro:panda_link lname="panda_leftfinger" vmesh="${mesh_pkg_visual}/finger.dae" cmesh="${mesh_pkg_collision}/finger.stl" color="panda_gray" mass="0.05" ixx="0.0005" iyy="0.0005" izz="0.0005"/>
-  <xacro:panda_link lname="panda_rightfinger" vmesh="${mesh_pkg_visual}/finger.dae" cmesh="${mesh_pkg_collision}/finger.stl" color="panda_gray" mass="0.05" ixx="0.0005" iyy="0.0005" izz="0.0005"/>
+  <xacro:panda_link lname="panda_link0" vmesh="${mesh_pkg_visual}/link0.dae" cmesh="${mesh_pkg_collision}/link0.stl" imesh="${link0_mesh}" color="panda_dark" mass="1.0" ixx="0.01" iyy="0.01" izz="0.01"/>
+  <xacro:panda_link lname="panda_link1" vmesh="${mesh_pkg_visual}/link1.dae" cmesh="${mesh_pkg_collision}/link1.stl" imesh="${link1_mesh}" color="panda_gray" mass="1.0" ixx="0.01" iyy="0.01" izz="0.01"/>
+  <xacro:panda_link lname="panda_link2" vmesh="${mesh_pkg_visual}/link2.dae" cmesh="${mesh_pkg_collision}/link2.stl" imesh="${link2_mesh}"  color="panda_white" mass="1.0" ixx="0.01" iyy="0.01" izz="0.01"/>
+  <xacro:panda_link lname="panda_link3" vmesh="${mesh_pkg_visual}/link3.dae" cmesh="${mesh_pkg_collision}/link3.stl" imesh="${link3_mesh}"  color="panda_gray" mass="1.0" ixx="0.01" iyy="0.01" izz="0.01"/>
+  <xacro:panda_link lname="panda_link4" vmesh="${mesh_pkg_visual}/link4.dae" cmesh="${mesh_pkg_collision}/link4.stl" imesh="${link4_mesh}"  color="panda_white" mass="1.0" ixx="0.01" iyy="0.01" izz="0.01"/>
+  <xacro:panda_link lname="panda_link5" vmesh="${mesh_pkg_visual}/link5.dae" cmesh="${mesh_pkg_collision}/link5.stl" imesh="${link5_mesh}"  color="panda_gray" mass="1.0" ixx="0.01" iyy="0.01" izz="0.01"/>
+  <xacro:panda_link lname="panda_link6" vmesh="${mesh_pkg_visual}/link6.dae" cmesh="${mesh_pkg_collision}/link6.stl" imesh="${link6_mesh}"  color="panda_white" mass="0.8" ixx="0.008" iyy="0.008" izz="0.008"/>
+  <xacro:panda_link lname="panda_link7" vmesh="${mesh_pkg_visual}/link7.dae" cmesh="${mesh_pkg_collision}/link7.stl" imesh="${link7_mesh}"  color="panda_dark" mass="0.6" ixx="0.006" iyy="0.006" izz="0.006"/>
+  <xacro:panda_link lname="panda_hand" vmesh="${mesh_pkg_visual}/hand.dae" cmesh="${mesh_pkg_collision}/hand.stl" imesh="${hand_mesh}"   color="panda_dark" mass="0.2" ixx="0.002" iyy="0.002" izz="0.002"/>
+  <xacro:panda_link lname="panda_leftfinger" vmesh="${mesh_pkg_visual}/finger.dae" cmesh="${mesh_pkg_collision}/finger.stl" imesh="${finger_mesh}"  color="panda_gray" mass="0.05" ixx="0.0005" iyy="0.0005" izz="0.0005"/>
+  <xacro:panda_link lname="panda_rightfinger" vmesh="${mesh_pkg_visual}/finger.dae" cmesh="${mesh_pkg_collision}/finger.stl" imesh="${finger_mesh}"  color="panda_gray" mass="0.05" ixx="0.0005" iyy="0.0005" izz="0.0005"/>
   <link name="panda_link8"/>
   <joint name="base_to_panda_mount" type="fixed">
