Commit message: added actuators to the model

File: src/panda_ros_simulation/urdf/props.urdf.xacro (robot description, xacro)
@@ -1,15 +1,15 @@
 <?xml version="1.0"?>
 <robot xmlns:xacro="http://www.ros.org/wiki/xacro">
-  <xacro:property name="link0_mesh" value="link0"/>
-  <xacro:property name="link1_mesh" value="link1"/>
-  <xacro:property name="link2_mesh" value="link2"/>
-  <xacro:property name="link3_mesh" value="link3"/>
-  <xacro:property name="link4_mesh" value="link4"/>
-  <xacro:property name="link5_mesh" value="link5"/>
-  <xacro:property name="link6_mesh" value="link6"/>
-  <xacro:property name="link7_mesh" value="link7"/>
-  <xacro:property name="hand_mesh" value="hand"/>
-  <xacro:property name="finger_mesh" value="finger"/>
-<xacro:macro name="panda_inertial" params="
+  <xacro:property name="link0_mesh" value="link0" />
+  <xacro:property name="link1_mesh" value="link1" />
+  <xacro:property name="link2_mesh" value="link2" />
+  <xacro:property name="link3_mesh" value="link3" />
+  <xacro:property name="link4_mesh" value="link4" />
+  <xacro:property name="link5_mesh" value="link5" />
+  <xacro:property name="link6_mesh" value="link6" />
+  <xacro:property name="link7_mesh" value="link7" />
+  <xacro:property name="hand_mesh" value="hand" />
+  <xacro:property name="finger_mesh" value="finger" />
+  <xacro:macro name="panda_inertial" params="
     mesh
     mesh_offset_rpy:=${mesh_offset_rpy}
@@ -17,72 +17,82 @@
     <xacro:if value="${mesh == link0_mesh}">
       <inertial>
-        <origin xyz="-0.025566 -2.87883e-05 0.057332" rpy="${mesh_offset_rpy}"/>
-        <mass value="2.814271300104062"/>
-        <inertia ixx="0.0075390636364814695" iyy="0.010508017427382959" izz="0.009864933638708275" ixy="-1.5053124574783335e-05" ixz="-0.0012144328835738973" iyz="1.0434803501032979e-05"/>
+        <origin xyz="-0.025566 -2.87883e-05 0.057332" rpy="${mesh_offset_rpy}" />
+        <mass value="2.814271300104062" />
+        <inertia ixx="0.0075390636364814695" iyy="0.010508017427382959" izz="0.009864933638708275"
+          ixy="-1.5053124574783335e-05" ixz="-0.0012144328835738973" iyz="1.0434803501032979e-05" />
       </inertial>
     </xacro:if>
     <xacro:if value="${mesh == link1_mesh}">
       <inertial>
-        <origin xyz="-3.72212e-09 -0.0324958 -0.0675818" rpy="${mesh_offset_rpy}"/>
-        <mass value="2.6433170427227215"/>
-        <inertia ixx="0.017405076982879724" iyy="0.015352077935781732" izz="0.005987891663073857" ixy="-8.687986369621078e-09" ixz="-1.6277819062920423e-08" iyz="0.004510855959102245"/>
+        <origin xyz="-3.72212e-09 -0.0324958 -0.0675818" rpy="${mesh_offset_rpy}" />
+        <mass value="2.6433170427227215" />
+        <inertia ixx="0.017405076982879724" iyy="0.015352077935781732" izz="0.005987891663073857"
+          ixy="-8.687986369621078e-09" ixz="-1.6277819062920423e-08" iyz="0.004510855959102245" />
       </inertial>
     </xacro:if>
     <xacro:if value="${mesh == link2_mesh}">
       <inertial>
-        <origin xyz="3.17833e-07 -0.06861 0.0322285" rpy="${mesh_offset_rpy}"/>
-        <mass value="2.6652755331661186"/>
-        <inertia ixx="0.01778694005635383" iyy="0.006044133867952844" izz="0.01571095500455695" ixy="8.70635625879119e-08" ixz="3.752072058394008e-08" iyz="-0.004599490295490376"/>
+        <origin xyz="3.17833e-07 -0.06861 0.0322285" rpy="${mesh_offset_rpy}" />
+        <mass value="2.6652755331661186" />
+        <inertia ixx="0.01778694005635383" iyy="0.006044133867952844" izz="0.01571095500455695"
+          ixy="8.70635625879119e-08" ixz="3.752072058394008e-08" iyz="-0.004599490295490376" />
       </inertial>
     </xacro:if>
     <xacro:if value="${mesh == link3_mesh}">
       <inertial>
-        <origin xyz="0.0469893 0.0316374 -0.031704" rpy="${mesh_offset_rpy}"/>
-        <mass value="2.3293714829045733"/>
-        <inertia ixx="0.0075496764161139766" iyy="0.009680676080191398" izz="0.007944557422008086" ixy="-0.0024320464513492225" ixz="-0.003250815048103007" iyz="-0.0021316282421730694"/>
+        <origin xyz="0.0469893 0.0316374 -0.031704" rpy="${mesh_offset_rpy}" />
+        <mass value="2.3293714829045733" />
+        <inertia ixx="0.0075496764161139766" iyy="0.009680676080191398" izz="0.007944557422008086"
+          ixy="-0.0024320464513492225" ixz="-0.003250815048103007" iyz="-0.0021316282421730694" />
       </inertial>
     </xacro:if>
     <xacro:if value="${mesh == link4_mesh}">
       <inertial>
-        <origin xyz="-0.0360505 0.0337069 0.0319019" rpy="${mesh_offset_rpy}"/>
-        <mass value="2.3104763646281508"/>
-        <inertia ixx="0.007764568814864828" iyy="0.008015776929980149" izz="0.009955882308071066" ixy="0.003371475204045935" ixz="-0.002343621113168248" iyz="0.0022917526161470624"/>
+        <origin xyz="-0.0360505 0.0337069 0.0319019" rpy="${mesh_offset_rpy}" />
+        <mass value="2.3104763646281508" />
+        <inertia ixx="0.007764568814864828" iyy="0.008015776929980149" izz="0.009955882308071066"
+          ixy="0.003371475204045935" ixz="-0.002343621113168248" iyz="0.0022917526161470624" />
       </inertial>
     </xacro:if>
     <xacro:if value="${mesh == link5_mesh}">
       <inertial>
-        <origin xyz="-6.12525e-06 0.0610427 -0.104176" rpy="${mesh_offset_rpy}"/>
-        <mass value="2.6226426154892004"/>
-        <inertia ixx="0.029070538014399377" iyy="0.027638529986528795" izz="0.004251111234400737" ixy="6.208738268725568e-07" ixz="-1.0059151925023392e-05" iyz="-0.007424306477850814"/>
+        <origin xyz="-6.12525e-06 0.0610427 -0.104176" rpy="${mesh_offset_rpy}" />
+        <mass value="2.6226426154892004" />
+        <inertia ixx="0.029070538014399377" iyy="0.027638529986528795" izz="0.004251111234400737"
+          ixy="6.208738268725568e-07" ixz="-1.0059151925023392e-05" iyz="-0.007424306477850814" />
       </inertial>
     </xacro:if>
     <xacro:if value="${mesh == link6_mesh}">
       <inertial>
-        <origin xyz="0.051051 0.00910797 0.0106343" rpy="${mesh_offset_rpy}"/>
-        <mass value="1.5025804886626795"/>
-        <inertia ixx="0.002940555801469018" iyy="0.00392105201248677" izz="0.0054115603870960195" ixy="-0.00042391108351381507" ixz="0.000610007735338717" iyz="0.00012647545430836214"/>
+        <origin xyz="0.051051 0.00910797 0.0106343" rpy="${mesh_offset_rpy}" />
+        <mass value="1.5025804886626795" />
+        <inertia ixx="0.002940555801469018" iyy="0.00392105201248677" izz="0.0054115603870960195"
+          ixy="-0.00042391108351381507" ixz="0.000610007735338717" iyz="0.00012647545430836214" />
       </inertial>
     </xacro:if>
     <xacro:if value="${mesh == link7_mesh}">
       <inertial>
-        <origin xyz="0.0109695 0.0107965 0.0650412" rpy="${mesh_offset_rpy}"/>
-        <mass value="0.5237668134788256"/>
-        <inertia ixx="0.0008621467959726535" iyy="0.0008613100184801048" izz="0.0006961139396618219" ixy="-0.00011871071570425467" ixz="3.866602604509339e-05" iyz="-9.057841649422724e-05"/>
+        <origin xyz="0.0109695 0.0107965 0.0650412" rpy="${mesh_offset_rpy}" />
+        <mass value="0.5237668134788256" />
+        <inertia ixx="0.0008621467959726535" iyy="0.0008613100184801048" izz="0.0006961139396618219"
+          ixy="-0.00011871071570425467" ixz="3.866602604509339e-05" iyz="-9.057841649422724e-05" />
       </inertial>
     </xacro:if>
     <xacro:if value="${mesh == hand_mesh}">
       <inertial>
-        <origin xyz="-6.7624e-06 0.00152435 0.0275912" rpy="${mesh_offset_rpy}"/>
-        <mass value="0.14060765127978503"/>
-        <inertia ixx="0.0005365450414352072" iyy="7.70511954783727e-05" izz="0.0004938176882694914" ixy="1.7911952957732454e-08" ixz="-2.320071910601251e-08" iyz="4.681149945315967e-08"/>
+        <origin xyz="-6.7624e-06 0.00152435 0.0275912" rpy="${mesh_offset_rpy}" />
+        <mass value="0.14060765127978503" />
+        <inertia ixx="0.0005365450414352072" iyy="7.70511954783727e-05" izz="0.0004938176882694914"
+          ixy="1.7911952957732454e-08" ixz="-2.320071910601251e-08" iyz="4.681149945315967e-08" />
       </inertial>
     </xacro:if>
     <xacro:if value="${mesh == finger_mesh}">
       <inertial>
-        <origin xyz="-6.2561e-06 0.00227781 -0.0277116" rpy="${mesh_offset_rpy}"/>
-        <mass value="0.2238453537819424"/>
-        <inertia ixx="6.74804167363695e-05" iyy="6.627189221641395e-05" izz="1.550396267804825e-05" ixy="-4.1027443646025676e-09" ixz="1.8693673970152995e-08" iyz="1.1967548474390802e-05"/>
+        <origin xyz="-6.2561e-06 0.00227781 -0.0277116" rpy="${mesh_offset_rpy}" />
+        <mass value="0.2238453537819424" />
+        <inertia ixx="6.74804167363695e-05" iyy="6.627189221641395e-05" izz="1.550396267804825e-05"
+          ixy="-4.1027443646025676e-09" ixz="1.8693673970152995e-08" iyz="1.1967548474390802e-05" />
       </inertial>
     </xacro:if>
-</xacro:macro>
+  </xacro:macro>
 </robot>

Commit message: Added ros2_control

File: src/panda_ros_simulation/urdf/panda.urdf.xacro (robot description, xacro)
@@ -1,6 +1,8 @@
 <?xml version="1.0"?>
 <robot name="franka_panda" xmlns:xacro="http://www.ros.org/wiki/xacro">
-  <xacro:property name="mesh_pkg_visual" value="file:///home/akhil/panda_ros_simulation/install/panda_ros_simulation/share/panda_ros_simulation/meshes/visual" />
-  <xacro:property name="mesh_pkg_collision" value="file:///home/akhil/panda_ros_simulation/install/panda_ros_simulation/share/panda_ros_simulation/meshes/collision" />
+  <xacro:property name="mesh_pkg_visual"
+    value="file:///home/akhil/panda_ros_simulation/install/panda_ros_simulation/share/panda_ros_simulation/meshes/visual" />
+  <xacro:property name="mesh_pkg_collision"
+    value="file:///home/akhil/panda_ros_simulation/install/panda_ros_simulation/share/panda_ros_simulation/meshes/collision" />
   <xacro:property name="mesh_pkg_description" value="package://panda_ros_simulation/urdf" />
   <xacro:include filename="$(find panda_ros_simulation)/urdf/macros.urdf.xacro" />
@@ -190,5 +192,5 @@
     finger_link2_name="panda_rightfinger"
   />
-  <!-- <ros2_control name="PandaSystem" type="system">
+  <ros2_control name="PandaSystem" type="system">
     <hardware>
       <plugin>gazebo_ros2_control/GazeboSystem</plugin>
@@ -197,5 +199,7 @@
       <command_interface name="position" />
       <command_interface name="velocity" />
-      <state_interface name="position" />
+      <state_interface name="position">
+        <param name="initial_value">0.0</param>
+      </state_interface>
       <state_interface name="velocity" />
     </joint>
@@ -203,5 +207,7 @@
       <command_interface name="position" />
       <command_interface name="velocity" />
-      <state_interface name="position" />
+      <state_interface name="position">
+        <param name="initial_value">0.0</param>
+      </state_interface>
       <state_interface name="velocity" />
     </joint>
@@ -209,5 +215,7 @@
       <command_interface name="position" />
       <command_interface name="velocity" />
-      <state_interface name="position" />
+      <state_interface name="position">
+        <param name="initial_value">0.0</param>
+      </state_interface>
       <state_interface name="velocity" />
     </joint>
@@ -215,5 +223,7 @@
       <command_interface name="position" />
       <command_interface name="velocity" />
-      <state_interface name="position" />
+      <state_interface name="position">
+        <param name="initial_value">0.0</param>
+      </state_interface>
       <state_interface name="velocity" />
     </joint>
@@ -221,5 +231,7 @@
       <command_interface name="position" />
       <command_interface name="velocity" />
-      <state_interface name="position" />
+      <state_interface name="position">
+        <param name="initial_value">0.0</param>
+      </state_interface>
       <state_interface name="velocity" />
     </joint>
@@ -227,5 +239,7 @@
       <command_interface name="position" />
       <command_interface name="velocity" />
-      <state_interface name="position" />
+      <state_interface name="position">
+        <param name="initial_value">2.122</param>
+      </state_interface>
       <state_interface name="velocity" />
     </joint>
@@ -233,27 +247,36 @@
       <command_interface name="position" />
       <command_interface name="velocity" />
-      <state_interface name="position" />
-      <state_interface name="velocity" />
-    </joint>
-    <joint name="panda_finger_joint1">
-      <command_interface name="position" />
-      <command_interface name="velocity" />
-      <state_interface name="position" />
-      <state_interface name="velocity" />
-    </joint>
-    <joint name="panda_finger_joint2">
-      <command_interface name="position" />
-      <command_interface name="velocity" />
-      <state_interface name="position" />
+      <state_interface name="position">
+        <param name="initial_value">0.0</param>
+      </state_interface>
+      <state_interface name="velocity" />
+    </joint>
+    <joint name="finger_joint1">
+      <command_interface name="position" />
+      <command_interface name="velocity" />
+      <state_interface name="position">
+        <param name="initial_value">0.022</param>
+      </state_interface>
       <state_interface name="velocity" />
     </joint>
   </ros2_control>
-  <gazebo>
-    <plugin filename="libgazebo_ros2_control.so" name="gazebo_ros2_control">
-      <robot_param>robot_description</robot_param>
-      <robot_param_node>robot_state_publisher</robot_param_node>
+<!-- Ignition enable -->
+  <!-- <gazebo>
+    <plugin filename="libgz_ros2_control-system.so"
+      name="gz_ros2_control::GazeboSimROS2ControlPlugin">
+      <parameters>$(find panda_ros_simulation)/config/controller.yaml</parameters>
     </plugin>
   </gazebo> -->
+  <!-- clasic pluigin -->
   <gazebo>
+    <plugin filename="libgazebo_ros2_control.so"
+      name="gazebo_ros2_control">
+      <robotNamespace>/</robotNamespace>
+      <robotSimType>gazebo_ros2_control/GazeboSystem</robotSimType>
+      <parameters>$(find panda_ros_simulation)/config/controller.yaml</parameters>
+    </plugin>
+  </gazebo>
+  <!-- no ros2_control -->
+  <!-- <gazebo>
     <plugin name="gazebo_ros_joint_state_publisher"
       filename="libgazebo_ros_joint_state_publisher.so">
@@ -269,4 +292,4 @@
       <joint_name>finger_joint2</joint_name>
     </plugin>
-  </gazebo>
+  </gazebo> -->
 </robot>

Commit message: moveit config fix

File: src/panda_ros_simulation/urdf/panda.urdf.xacro (robot description, xacro)
@@ -23,10 +23,4 @@
   <xacro:property name="panda_green" value="Gazebo/Green" />
   <link name="world" />
-  <link name="base_link" />
-  <joint name="world_to_base" type="fixed">
-    <parent link="world" />
-    <child link="base_link" />
-    <origin xyz="0 0 0" rpy="0 0 0" />
-  </joint>
   <xacro:panda_link lname="panda_link0" vmesh="${mesh_pkg_visual}/link0.dae"
     cmesh="${mesh_pkg_collision}/link0.stl" imesh="${link0_mesh}" color="panda_dark" rgba_val="${panda_dark}"/>
@@ -115,5 +109,5 @@
   <xacro:property name="joint7_damping" value="3.0" />
   <xacro:property name="joint7_friction" value="0.48" />
-  <xacro:panda_joint parent="base_link" child="panda_link0" joint_name="base_to_panda_mount"
+  <xacro:panda_joint parent="world" child="panda_link0" joint_name="base_to_panda_mount"
     joint_type="fixed" joint_origin_xyz="0 0 0" joint_origin_rpy="0 0 0" />
   <!-- 1st -->

Commit message: Adding eef single finger working

File: src/panda_ros_simulation/urdf/panda.urdf.xacro (robot description, xacro)
@@ -24,25 +24,36 @@
   <link name="world" />
   <xacro:panda_link lname="panda_link0" vmesh="${mesh_pkg_visual}/link0.dae"
-    cmesh="${mesh_pkg_collision}/link0.stl" imesh="${link0_mesh}" color="panda_dark" rgba_val="${panda_dark}"/>
+    cmesh="${mesh_pkg_collision}/link0.stl" imesh="${link0_mesh}" color="panda_dark"
+    rgba_val="${panda_dark}" />
   <xacro:panda_link lname="panda_link1" vmesh="${mesh_pkg_visual}/link1.dae"
-    cmesh="${mesh_pkg_collision}/link1.stl" imesh="${link1_mesh}" color="panda_gray" rgba_val= "${panda_gray}"/>
+    cmesh="${mesh_pkg_collision}/link1.stl" imesh="${link1_mesh}" color="panda_gray"
+    rgba_val="${panda_gray}" />
   <xacro:panda_link lname="panda_link2" vmesh="${mesh_pkg_visual}/link2.dae"
-    cmesh="${mesh_pkg_collision}/link2.stl" imesh="${link2_mesh}" color="panda_white" rgba_val="${panda_white}"/>
+    cmesh="${mesh_pkg_collision}/link2.stl" imesh="${link2_mesh}" color="panda_white"
+    rgba_val="${panda_white}" />
   <xacro:panda_link lname="panda_link3" vmesh="${mesh_pkg_visual}/link3.dae"
-    cmesh="${mesh_pkg_collision}/link3.stl" imesh="${link3_mesh}" color="panda_gray" rgba_val="${panda_gray}"/>
+    cmesh="${mesh_pkg_collision}/link3.stl" imesh="${link3_mesh}" color="panda_gray"
+    rgba_val="${panda_gray}" />
   <xacro:panda_link lname="panda_link4" vmesh="${mesh_pkg_visual}/link4.dae"
-    cmesh="${mesh_pkg_collision}/link4.stl" imesh="${link4_mesh}" color="panda_white" rgba_val="${panda_white}"/>
+    cmesh="${mesh_pkg_collision}/link4.stl" imesh="${link4_mesh}" color="panda_white"
+    rgba_val="${panda_white}" />
   <xacro:panda_link lname="panda_link5" vmesh="${mesh_pkg_visual}/link5.dae"
-    cmesh="${mesh_pkg_collision}/link5.stl" imesh="${link5_mesh}" color="panda_gray" rgba_val= "${panda_gray}"/>
+    cmesh="${mesh_pkg_collision}/link5.stl" imesh="${link5_mesh}" color="panda_gray"
+    rgba_val="${panda_gray}" />
   <xacro:panda_link lname="panda_link6" vmesh="${mesh_pkg_visual}/link6.dae"
-    cmesh="${mesh_pkg_collision}/link6.stl" imesh="${link6_mesh}" color="panda_white" rgba_val="${panda_white}" />
+    cmesh="${mesh_pkg_collision}/link6.stl" imesh="${link6_mesh}" color="panda_white"
+    rgba_val="${panda_white}" />
   <xacro:panda_link lname="panda_link7" vmesh="${mesh_pkg_visual}/link7.dae"
-    cmesh="${mesh_pkg_collision}/link7.stl" imesh="${link7_mesh}" color="panda_dark" rgba_val="${panda_dark}"/>
+    cmesh="${mesh_pkg_collision}/link7.stl" imesh="${link7_mesh}" color="panda_dark"
+    rgba_val="${panda_dark}" />
   <xacro:panda_link lname="panda_hand" vmesh="${mesh_pkg_visual}/hand.dae"
-    cmesh="${mesh_pkg_collision}/hand.stl" imesh="${hand_mesh}" color="panda_dark" rgba_val="${panda_dark}" />
+    cmesh="${mesh_pkg_collision}/hand.stl" imesh="${hand_mesh}" color="panda_dark"
+    rgba_val="${panda_dark}" />
   <xacro:panda_link lname="panda_leftfinger" vmesh="${mesh_pkg_visual}/finger.dae"
-    cmesh="${mesh_pkg_collision}/finger.stl" imesh="${finger_mesh}" color="panda_gray" rgba_val="${panda_green}"/>
+    cmesh="${mesh_pkg_collision}/finger.stl" imesh="${finger_mesh}" color="panda_gray"
+    rgba_val="${panda_green}" />
   <xacro:panda_link lname="panda_rightfinger" vmesh="${mesh_pkg_visual}/finger.dae"
-    cmesh="${mesh_pkg_collision}/finger.stl" imesh="${finger_mesh}" color="panda_gray" rgba_val="${panda_green}"/>
+    cmesh="${mesh_pkg_collision}/finger.stl" imesh="${finger_mesh}" color="panda_gray"
+    rgba_val="${panda_green}" />
   <link name="panda_link8" />
   <xacro:property name="joint1_origin_xyz" value="0 0 0.333" />
@@ -252,5 +263,4 @@
     <joint name="finger_joint1">
       <command_interface name="position" />
-      <command_interface name="velocity" />
       <state_interface name="position">
         <param name="initial_value">0.022</param>
@@ -258,6 +268,13 @@
       <state_interface name="velocity" />
     </joint>
+    <joint name="finger_joint2">
+      <command_interface name="position" />
+      <state_interface name="position">
+        <param name="initial_value">0.0</param>
+      </state_interface>
+      <state_interface name="velocity" />
+    </joint>
   </ros2_control>
-<!-- Ignition enable -->
+  <!-- Ignition enable -->
   <!-- <gazebo>
     <plugin filename="libgz_ros2_control-system.so"
